File: 3d_tree_pyramid_base.kicad_pcb (KiCad board)
At the start: 2 copper layers, 60 x 60 mm, 16 parts, among them J1 USB4125, J2 +5V, J3 +5V, J4 GND, J5 GND, Q1 DMG2302U, SW1 SW_SPDT

Commit message: Update to taller cone
Routing:
- net /SGND: track 77.5 -> 78.1 mm
Other:
- board text added: "v0.0.1 10/30/21"
- board text removed: "v0.0.1 10/12/21"
