File: 3d_tree_pyramid_control.kicad_pcb (KiCad board)
At the start: 2 copper layers, 21 x 51 mm, 22 parts, among them J1 Conn, J2 Conn, J3 Conn, J4 Conn, J5 AVR-ISP-6, J6 Conn, J7 Conn, J8 Conn, J9 Conn, U1 ATtiny461A-XU

Commit message: Update to taller cone
Parts:
- moved D1 25.4 mm to (40.5, 87.0)
- moved D2 12.2 mm to (37.0, 107.0)
- moved D3 8.36 mm to (44.0, 116.0)
- moved D4 7.53 mm to (36.0, 124.0)
- moved D6 6.47 mm to (35.5, 139.4)
- moved D5 5.37 mm to (45.5, 133.0)
- moved REF** 5.20 mm to (40.6, 107.4)
- moved D7 3.99 mm to (47.0, 147.0)
- moved J5 1.20 mm to (40.4, 120.3)
Connections:
- U1 pad 11: (no net) -> Net-(U1-Pad11)
- U1 pad 12: (no net) -> Net-(U1-Pad12)
- U1 pad 13: (no net) -> Net-(U1-Pad13)
- U1 pad 14: (no net) -> Net-(U1-Pad14)
- U1 pad 17: (no net) -> Net-(U1-Pad17)
- U1 pad 18: (no net) -> Net-(U1-Pad18)
- U1 pad 19: (no net) -> Net-(U1-Pad19)
- U1 pad 4: (no net) -> Net-(U1-Pad4)
- U1 pad 7: (no net) -> Net-(U1-Pad7)
- U1 pad 8: (no net) -> Net-(U1-Pad8)
- U1 pad 9: (no net) -> Net-(U1-Pad9)
Routing:
- net /DINT: track 34.6 -> 65.3 mm
- net /+5V: track 127.0 -> 146.2 mm, vias 5 -> 8
- net /SCK: track 30.6 -> 17.1 mm
- net Net-(D1-Pad1): track 8.69 -> 20.9 mm
- net /GND: track 14.8 -> 8.36 mm, vias 27 -> 31
- net /MISO: track 23.7 -> 17.4 mm, vias 2 -> 0
- net /MOSI: track 25.3 -> 20.0 mm, vias 2 -> 0
- net /~RST: track 19.0 -> 22.6 mm, vias 0 -> 2
- net Net-(D4-Pad1): track 16.0 -> 12.7 mm
- net Net-(D6-Pad1): track 16.0 -> 13.3 mm, vias 2 -> 0
- net Net-(D3-Pad1): track 17.4 -> 14.9 mm
- net Net-(D5-Pad1): track 18.6 -> 17.0 mm
- net /DOUT: track 19.3 -> 18.1 mm
Other:
- board size 21 x 51 mm -> 21 x 91 mm
- board text added: "v0.0.1 10/30/21"
- board text removed: "v0.0.0 09/22/21"
