File: 3d_tree_pyramid_control.sch (KiCad schematic (older format))
At the start: 21 parts, among them J1 Conn, J2 Conn, J3 Conn, J4 Conn, J5 AVR-ISP-6, J6 Conn, J7 Conn, J8 Conn, J9 Conn, U1 ATtiny461A-XU

Commit message: Update to taller cone
Parts:
- J5: footprint WM_lib:Hirose_DF23C-20DP-ISP6 -> WM_lib:pogo_pads_2x03_p2.54mm
Changed lines of the file:
@@
 F 0 "J5" H 1121 4896 50  0000 R CNN
 F 1 "AVR-ISP-6" H 1121 4805 50  0000 R CNN
-F 2 "WM_lib:Hirose_DF23C-20DP-ISP6" V 1200 4850 50  0001 C CNN
+F 2 "WM_lib:pogo_pads_2x03_p2.54mm" V 1200 4850 50  0001 C CNN
 F 3 " ~" H 175 4250 50  0001 C CNN
 	1    1450 4800
