File: 3d_tree_pyramid_display.kicad_pcb (KiCad board)
At the start: 2 copper layers, 21 x 51 mm, 15 parts, among them J1 Conn, J2 Conn, J3 Conn, J4 Conn, J5 Conn, J6 Conn

Commit message: Update to taller cone
Parts:
- moved D1 25.4 mm to (40.5, 87.0)
- moved D2 12.2 mm to (37.0, 107.0)
- moved D3 8.36 mm to (44.0, 116.0)
- moved D4 7.53 mm to (36.0, 124.0)
- moved D6 6.47 mm to (35.5, 139.4)
- moved D5 5.37 mm to (45.5, 133.0)
- moved REF** 4.30 mm to (44.9, 126.2)
- moved D7 3.99 mm to (47.0, 147.0)
- moved C1 0.80 mm to (39.7, 132.0), turned to 0 degrees
Routing:
- net /DIN: track 45.4 -> 70.4 mm, vias 3 -> 1
- net Net-(D1-Pad1): track 10.7 -> 20.9 mm
- net /+5V: track 96.7 -> 102.5 mm, vias 5 -> 7
- net Net-(D5-Pad1): track 17.8 -> 14.4 mm
- net Net-(D4-Pad1): track 14.9 -> 11.9 mm
- net Net-(D6-Pad1): track 16.0 -> 13.3 mm
- net Net-(D3-Pad1): track 15.2 -> 12.9 mm
- net /DOUT: track 18.2 -> 16.5 mm
- net /GND: track 1.78 -> 2.95 mm, vias 14 -> 24
Other:
- board size 21 x 51 mm -> 21 x 91 mm
- board text added: "v0.0.1 10/29/21"
- board text removed: "v0.0.0 09/24/21"
